File: eagle/segmentring4und8.sch (EAGLE design)
At the start: 12 parts

Commit message: Schaltpläne fertig
Connections:
- net E1 renamed N$4
- net E2 renamed N$5
- net E3 renamed N$6
- net E4 renamed N$7
- removed net 1: 1.MP
- removed net 2: 2.MP
- removed net 3: 3.MP
- removed net 4: 4.MP
- removed net 5: 5.MP
- removed net 6: 6.MP
- removed net 7: 7.MP
- removed net 8: 8.MP
Changed lines of the file:
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@@
 </busses>
 <nets>
-<net name="E1" class="0">
+<net name="N$4" class="0">
 <segment>
 <pinref part="E1" gate="1" pin="MP"/>
@@
 </segment>
 </net>
-<net name="E2" class="0">
+<net name="N$5" class="0">
 <segment>
 <pinref part="E2" gate="1" pin="MP"/>
@@
 </segment>
 </net>
-<net name="E3" class="0">
+<net name="N$6" class="0">
 <segment>
 <pinref part="E3" gate="1" pin="MP"/>
@@
 </segment>
 </net>
-<net name="E4" class="0">
+<net name="N$7" class="0">
 <segment>
 <pinref part="E4" gate="1" pin="MP"/>
@@
 </segment>
 </net>
-<net name="7" class="0">
-<segment>
-<pinref part="7" gate="1" pin="MP"/>
-<wire x1="93.98" y1="35.56" x2="93.98" y2="38.1" width="0.1524" layer="91"/>
-</segment>
-</net>
-<net name="8" class="0">
-<segment>
-<pinref part="8" gate="1" pin="MP"/>
-<wire x1="101.6" y1="35.56" x2="101.6" y2="38.1" width="0.1524" layer="91"/>
-</segment>
-</net>
-<net name="5" class="0">
-<segment>
-<pinref part="5" gate="1" pin="MP"/>
-<wire x1="111.76" y1="35.56" x2="111.76" y2="38.1" width="0.1524" layer="91"/>
-</segment>
-</net>
-<net name="6" class="0">
-<segment>
-<pinref part="6" gate="1" pin="MP"/>
-<wire x1="121.92" y1="35.56" x2="121.92" y2="38.1" width="0.1524" layer="91"/>
-</segment>
-</net>
-<net name="3" class="0">
-<segment>
-<pinref part="3" gate="1" pin="MP"/>
-<wire x1="132.08" y1="35.56" x2="132.08" y2="38.1" width="0.1524" layer="91"/>
-</segment>
-</net>
-<net name="4" class="0">
-<segment>
-<pinref part="4" gate="1" pin="MP"/>
-<wire x1="142.24" y1="35.56" x2="142.24" y2="38.1" width="0.1524" layer="91"/>
-</segment>
-</net>
-<net name="1" class="0">
-<segment>
-<pinref part="1" gate="1" pin="MP"/>
-<wire x1="152.4" y1="35.56" x2="152.4" y2="38.1" width="0.1524" layer="91"/>
-</segment>
-</net>
-<net name="2" class="0">
-<segment>
-<pinref part="2" gate="1" pin="MP"/>
-<wire x1="165.1" y1="35.56" x2="165.1" y2="38.1" width="0.1524" layer="91"/>
-</segment>
-</net>
