File: eagle/segmentring4und8klein.brd (EAGLE design)
At the start: 100 x 150 mm, 12 parts

Commit message: Schaltpläne fertig
Parts:
- moved 2 3.86 mm to (80.6, 31.8)
- moved 1 3.86 mm to (76.8, 31.8)
- moved 4 2.62 mm to (80.6, 27.9)
- moved 3 2.62 mm to (76.8, 27.9)
- moved 6 1.42 mm to (80.6, 24.1)
- moved 5 1.42 mm to (76.8, 24.1)
- moved 8 0.64 mm to (80.6, 20.3)
- moved 7 0.63 mm to (76.8, 20.3)
Connections:
- net E1 renamed N$4
- net E2 renamed N$5
- net E3 renamed N$6
- net E4 renamed N$7
- removed net 1: 1.MP
- removed net 2: 2.MP
- removed net 3: 3.MP
- removed net 4: 4.MP
- removed net 5: 5.MP
- removed net 6: 6.MP
- removed net 7: 7.MP
- removed net 8: 8.MP
Routing:
- net S$3: track 0.00 -> 137.6 mm
- net E1: track 0.00 -> 110.2 mm, vias 0 -> 1
- net N$5: track 105.1 -> 0.00 mm, vias 1 -> 0
- net E3: track 0.00 -> 99.4 mm, vias 0 -> 1
- net N$4: track 96.9 -> 0.00 mm, vias 1 -> 0
- net N$7: track 94.5 -> 0.00 mm, vias 1 -> 0
- net E2: track 0.00 -> 93.2 mm, vias 0 -> 1
- net N$6: track 86.9 -> 0.00 mm, vias 1 -> 0
- net E4: track 0.00 -> 81.6 mm, vias 0 -> 1
- net N$2: track 77.0 -> 0.00 mm
- net S$1: track 0.00 -> 68.1 mm
- net N$1: track 57.1 -> 0.00 mm
- net N$3: track 27.9 -> 0.00 mm
- net 2: track 75.1 -> 99.7 mm
- net 1: track 75.1 -> 99.1 mm
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- added copper zone on layer 1, net E1
- added copper zone on layer 1, net E2
- added copper zone on layer 1, net E3
- added copper zone on layer 1, net E4
- added copper zone on layer 16, net N$8
- removed copper zone on layer 1, net N$4
- removed copper zone on layer 1, net N$5
- removed copper zone on layer 1, net N$6
- removed copper zone on layer 1, net N$7

Commit message: Verbesserung der Boards
Connections:
- new net 1: 1.MP
- new net 2: 2.MP
- new net 3: 3.MP
- new net 4: 4.MP
- new net 5: 5.MP
- new net 6: 6.MP
- new net 7: 7.MP
- new net 8: 8.MP
Routing:
- net S$3: track 137.6 -> 93.0 mm
- net S$4: track 0.00 -> 30.1 mm
- net 2: track 99.7 -> 81.8 mm
- net 1: track 99.1 -> 81.8 mm
- net 7: track 108.0 -> 115.4 mm
- net 5: track 97.7 -> 104.9 mm
- net 6: track 98.2 -> 105.0 mm
- net 8: track 108.7 -> 115.4 mm
- net 3: track 86.9 -> 93.0 mm
- net 4: track 87.3 -> 92.9 mm
- net E3: track 99.4 -> 100.9 mm
- net E1: track 110.2 -> 111.0 mm
- net E4: track 81.6 -> 82.3 mm
- removed copper zone on layer 16, net GND
- removed copper zone on layer 16, net N$8

Commit message: bessere Linien
Routing:
- net S$1: track 68.1 -> 33.5 mm
- net S$5: track 0.00 -> 15.8 mm
Changed lines of the file:
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@@
 </signal>
 <signal name="E4">
-<via x="39" y="113" extent="1-16" drill="0.6" shape="square"/>
+<via x="39" y="113" extent="1-16" drill="0.6" diameter="0.254" shape="square"/>
 <wire x1="33.6" y1="109.8" x2="39" y2="113" width="0.6096" layer="16" curve="20.505911"/>
 <wire x1="33.6" y1="109.8" x2="33.6" y2="35.6" width="0.6096" layer="16"/>
@@
 <contactref element="E4" pad="MP"/>
 </signal>
+<signal name="S$5">
+<wire x1="31.7" y1="120.7" x2="31.7" y2="136.5" width="0" layer="1"/>
+</signal>
 <signal name="S$1">
-<wire x1="46.5" y1="120.8" x2="13" y2="120.8" width="0.4064" layer="1"/>
-<wire x1="13" y1="120.8" x2="13" y2="120.7" width="0.4064" layer="1"/>
-<wire x1="13" y1="120.7" x2="31.7" y2="120.7" width="0.4064" layer="1"/>
-<wire x1="31.7" y1="120.7" x2="31.7" y2="136.5" width="0.4064" layer="1"/>
+<wire x1="46.5" y1="120.8" x2="13" y2="120.8" width="0" layer="1"/>
 </signal>
 <signal name="S$2">
-<wire x1="31.8" y1="120.7" x2="31.8" y2="104.8" width="0.4064" layer="1"/>
+<wire x1="31.8" y1="120.7" x2="31.8" y2="104.8" width="0" layer="1"/>
 </signal>
 <signal name="S$4">
-<wire x1="89.1" y1="130.9" x2="89" y2="130.9" width="0.4064" layer="1"/>
-<wire x1="89" y1="130.9" x2="67.8" y2="109.7" width="0.4064" layer="1"/>
+<wire x1="89" y1="130.9" x2="67.8" y2="109.7" width="0" layer="1"/>
 </signal>
 <signal name="S$3">
-<wire x1="78.8" y1="134.7" x2="78.8" y2="120.6" width="0.4064" layer="1"/>
-<wire x1="78.8" y1="105.6" x2="78.8" y2="120.6" width="0.4064" layer="1"/>
-<wire x1="78.8" y1="120.6" x2="95" y2="120.6" width="0.4064" layer="1"/>
-<wire x1="60.8" y1="120.6" x2="78.8" y2="120.6" width="0.4064" layer="1"/>
-<wire x1="78.8" y1="120.6" x2="89.4" y2="110" width="0.4064" layer="1"/>
-<wire x1="78.8" y1="120.6" x2="68.4" y2="131" width="0.4064" layer="1"/>
+<wire x1="78.8" y1="134.7" x2="78.8" y2="120.6" width="0" layer="1"/>
+<wire x1="78.8" y1="105.6" x2="78.8" y2="120.6" width="0" layer="1"/>
+<wire x1="78.8" y1="120.6" x2="95" y2="120.6" width="0" layer="1"/>
+<wire x1="60.8" y1="120.6" x2="78.8" y2="120.6" width="0" layer="1"/>
+<wire x1="78.8" y1="120.6" x2="89.4" y2="110" width="0" layer="1"/>
+<wire x1="78.8" y1="120.6" x2="68.4" y2="131" width="0" layer="1"/>
 </signal>
 </signals>
