File: eagle/segmentring4und8groß.brd (EAGLE design)
At the start: 150 x 150 mm, 12 parts

Commit message: Verbesserung der Boards
Routing:
- net 8: track 113.5 -> 116.3 mm
- net 4: track 82.9 -> 81.2 mm
- net 3: track 82.9 -> 81.2 mm
- net 7: track 114.0 -> 115.6 mm
- net E1: track 116.0 -> 117.0 mm
- net E3: track 104.5 -> 105.5 mm
- removed copper zone on layer 16, net GND
- removed copper zone on layer 16, net N$8

Commit message: bessere Linien
Changed lines of the file:
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@@
 </signal>
 <signal name="N$1">
-<wire x1="3.52" y1="120.76" x2="31.75" y2="120.65" width="0.4064" layer="1"/>
-<wire x1="56.84" y1="120.65" x2="31.75" y2="120.65" width="0.4064" layer="1"/>
-<wire x1="31.75" y1="120.65" x2="31.75" y2="148.14" width="0.4064" layer="1"/>
-<wire x1="31.75" y1="120.65" x2="31.65" y2="96.83" width="0.4064" layer="1"/>
+<wire x1="3.52" y1="120.76" x2="31.75" y2="120.65" width="0" layer="1"/>
+<wire x1="56.84" y1="120.65" x2="31.75" y2="120.65" width="0" layer="1"/>
+<wire x1="31.75" y1="120.65" x2="31.75" y2="148.14" width="0" layer="1"/>
+<wire x1="31.75" y1="120.65" x2="31.65" y2="96.83" width="0" layer="1"/>
 </signal>
 <signal name="N$4">
@@
 </signal>
 <signal name="N$2">
-<wire x1="69.98" y1="120.99" x2="98.21" y2="120.88" width="0.4064" layer="1"/>
-<wire x1="123.3" y1="120.88" x2="98.21" y2="120.88" width="0.4064" layer="1"/>
-<wire x1="98.21" y1="120.88" x2="98.21" y2="148.37" width="0.4064" layer="1"/>
-<wire x1="98.21" y1="120.88" x2="98.11" y2="97.06" width="0.4064" layer="1"/>
+<wire x1="69.98" y1="120.99" x2="98.21" y2="120.88" width="0" layer="1"/>
+<wire x1="123.3" y1="120.88" x2="98.21" y2="120.88" width="0" layer="1"/>
+<wire x1="98.21" y1="120.88" x2="98.21" y2="148.37" width="0" layer="1"/>
+<wire x1="98.21" y1="120.88" x2="98.11" y2="97.06" width="0" layer="1"/>
 </signal>
 <signal name="S$2">
-<wire x1="98.28" y1="120.9" x2="80.41" y2="138.77" width="0.4064" layer="1"/>
-<wire x1="80.41" y1="138.77" x2="80.41" y2="138.83" width="0.4064" layer="1"/>
+<wire x1="98.28" y1="120.9" x2="80.41" y2="138.77" width="0" layer="1"/>
 </signal>
 <signal name="S$3">
-<wire x1="98.17" y1="120.89" x2="116.37" y2="102.69" width="0.4064" layer="1"/>
-<wire x1="116.37" y1="102.69" x2="116.46" y2="102.69" width="0.4064" layer="1"/>
+<wire x1="98.17" y1="120.89" x2="116.37" y2="102.69" width="0" layer="1"/>
 </signal>
 <signal name="S$4">
-<wire x1="80.61" y1="103.32" x2="80.61" y2="103.09" width="0.4064" layer="1"/>
-<wire x1="80.61" y1="103.32" x2="116.35" y2="139.06" width="0.4064" layer="1"/>
+<wire x1="80.61" y1="103.32" x2="116.35" y2="139.06" width="0" layer="1"/>
 </signal>
 </signals>

Commit message: lawlz heavy
Parts:
- moved 1 12.1 mm to (96.1, 44.1)
- moved 2 12.1 mm to (99.9, 44.1)
- moved 7 12.1 mm to (96.1, 32.6)
- moved 8 12.1 mm to (99.9, 32.6)
- moved 3 12.1 mm to (96.1, 40.3)
- moved 4 12.1 mm to (99.9, 40.3)
- moved 5 12.1 mm to (96.1, 36.5)
- moved 6 12.1 mm to (99.9, 36.5)
Routing:
- net 3: track 81.2 -> 69.2 mm
- net 6: track 98.4 -> 86.3 mm
- net 5: track 99.3 -> 87.2 mm
- net 4: track 81.2 -> 69.2 mm
- net 1: track 106.5 -> 94.4 mm
- net 8: track 116.3 -> 104.2 mm
- net 7: track 115.6 -> 103.6 mm
- net 2: track 106.5 -> 94.5 mm
